File: addressable-haptics.sch (KiCad schematic (older format))
At the start: 8 parts, among them J1 Conn_01x02, J2 Conn_01x03, J3 Conn_01x03, J4 SOICBite, Q1 Q_PMOS_GSD, U1 ATtiny10-TS

Commit message: Update PCB
Parts:
- removed Q1: Q_PMOS_GSD, Package_TO_SOT_SMD:SOT-23, symbol Device:Q_PMOS_GSD
- added Q1: Q_PNP_BEC, Package_TO_SOT_SMD:SOT-23, symbol Device:Q_PNP_BEC
Connections:
- net 3.3V: now also Q1.2 (E)
- net signal_in: now also U1.4 (PB2); no longer J4.6 (Pin_6), U1.1 (PB0)
- net signal_out: now also J4.6 (Pin_6), U1.1 (PB0); no longer U1.4 (PB2)
- net to_motor: now also Q1.3 (C)
- net at R1.1: now also Q1.1 (B)
Changed lines of the file:
@@
 	0    1    1    0
-$EndComp
-$Comp
-L Device:Q_PMOS_GSD Q1
-U 1 1 5E4DD596
-P 5000 1650
-F 0 "Q1" H 5205 1696 50  0000 L CNN
-F 1 "Q_PMOS_GSD" H 5205 1605 50  0000 L CNN
-F 2 "Package_TO_SOT_SMD:SOT-23" H 5200 1750 50  0001 C CNN
-F 3 "~" H 5000 1650 50  0001 C CNN
-	1    5000 1650
-	1    0    0    -1
 $EndComp
 Wire Wire Line
@@
 Text Label 5050 4325 0    50   ~ 0
 tpi_rst
+Text Label 5475 2750 0    50   ~ 0
+signal_in
 Text Label 5475 2550 0    50   ~ 0
-signal_in
-Text Label 5475 2750 0    50   ~ 0
 signal_out
+$Comp
+L Device:Q_PNP_BEC Q1
+U 1 1 5F404B6A
+P 5000 1650
+F 0 "Q1" H 5225 1700 50  0000 L CNN
+F 1 "Q_PNP_BEC" H 5225 1650 50  0000 L CNN
+F 2 "Package_TO_SOT_SMD:SOT-23" H 5200 1750 50  0001 C CNN
+F 3 "~" H 5000 1650 50  0001 C CNN
+	1    5000 1650
+	1    0    0    -1
+$EndComp
 $EndSCHEMATC

Commit message: Fixed schematic
Parts:
- removed Q1: Q_PNP_BEC, Package_TO_SOT_SMD:SOT-23, symbol Device:Q_PNP_BEC
- added Q1: Q_NMOS_GSD, Package_TO_SOT_SMD:SOT-23, symbol Device:Q_NMOS_GSD
Connections:
- net 3.3V: now also Q1.3 (D)
- net to_motor: now also Q1.2 (S)
- net at R1.1: now also Q1.1 (G)
Changed lines of the file:
@@
 signal_out
 $Comp
-L Device:Q_PNP_BEC Q1
-U 1 1 5F404B6A
+L Device:Q_NMOS_GSD Q1
+U 1 1 5F48D374
 P 5000 1650
-F 0 "Q1" H 5225 1700 50  0000 L CNN
-F 1 "Q_PNP_BEC" H 5225 1650 50  0000 L CNN
+F 0 "Q1" H 5250 1600 50  0000 L CNN
+F 1 "Q_NMOS_GSD" H 5250 1650 50  0000 L CNN
 F 2 "Package_TO_SOT_SMD:SOT-23" H 5200 1750 50  0001 C CNN
 F 3 "~" H 5000 1650 50  0001 C CNN
 	1    5000 1650
-	1    0    0    -1
+	1    0    0    1
 $EndComp
 $EndSCHEMATC
